Commit message: Completed URDF Course

File: URDF/my_mira_description/urdf/mira_only_daes.urdf (robot description, URDF)
Before this commit: robot mira, 8 links, 7 joints
Links:
- link base_link: geometry visual mesh filename=package://my_mira_description/models/mira/meshes/mira_body_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
- link head_link: geometry visual mesh filename=package://my_mira_description/models/mira/meshes/mira_head_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
- link left_eye_link: geometry visual mesh filename=package://my_mira_description/models/mira/meshes/mira_eye_v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
- link right_eye_link: geometry visual mesh filename=package://my_mira_description/models/mira/meshes/mira_eye_v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
Joints:
- joint base_head_joint: origin xyz=0 0 0.06 rpy=0 0 0 -> xyz=0 0 0 rpy=0 0 0

Commit message: Learning Gazebo Simulator

File: URDF/my_mira_description/urdf/mira_only_daes.urdf (robot description, URDF)
Before this commit: robot mira, 8 links, 7 joints
Links:
- link roll_M1_link: mass None -> 0.001
